Commit message: fix: RS gravity compensation, add simulation packages and fake driver
Gravity compensation fix (hardware_manager.py):
- Remove non-blocking lock in gravity compensation tick to prevent
  skipped control cycles when the lock is contended
- Change request_feedback from True to False to avoid unnecessary
  CAN read latency during compensation
- Add gripper MIT mode initialization in enable()
- Send gripper MIT commands during gravity compensation to keep
  the gripper motor synchronized
- Lower gravity compensation kd from 1.5 to 1.0
- Remove tau_scale override (use default 1.0 for all joints)

Simulation support:
- Add fake_rs_driver.py: in-process fake motor driver for simulation
- Add fake_rs_bringup.launch.py: launch file for fake RS driver
- Add FakeRsDriver entry point in setup.py
- Add rebotarm_mujoco_rs package: MuJoCo physics sync, scene camera,
  color block detector, and task server for RS simulation
- Add rebotarm_agent package: MCP server and text agent for RS

Bringup updates:
- Add rosbridge_server exec_depend for web control
- Update 00-arm-rs_asm-v3.urdf with named materials and colors
- Add Seeed badge STL meshes
- Update rebotarm_hardware.yaml: kd 1.5 -> 1.0, remove tau_scale

File: src/rebotarm_bringup/description/urdf/00-arm-rs_asm-v3.urdf (robot description, URDF)
Before this commit: robot 00-arm-rs_asm-v3, 10 links, 9 joints
Links:
- link link3: geometry collision mesh filename=package://rebotarm_bringup/description/meshes_rs/link3.STL; visual mesh filename=package://rebotarm_bringup/description/meshes_rs/cnc3.STL
