Commit message: Add DM and RS URDF and MoveIt integration

File: src/rebotarm_moveit_config/config/rebotarm.urdf.xacro (robot description, xacro)
@@ -1,11 +1,11 @@
 <?xml version="1.0"?>
-<robot xmlns:xacro="http://www.ros.org/wiki/xacro" name="reBot_B601_DM_with_gripper">
+<robot xmlns:xacro="http://www.ros.org/wiki/xacro" name="ReBot_Arm_DM">
   <xacro:arg name="initial_positions_file" default="$(find rebotarm_moveit_config)/config/initial_positions.yaml"/>
-  <xacro:include filename="$(find rebotarm_bringup)/description/urdf/reBot_B601_DM_with_gripper.urdf"/>
+  <xacro:include filename="$(find rebotarm_bringup)/description/DM/urdf/ReBot_Arm_DM.urdf"/>
   <xacro:include filename="$(find rebotarm_moveit_config)/config/rebotarm.ros2_control.xacro"/>
   <link name="gripper_tcp"/>
   <joint name="gripper_tcp_joint" type="fixed">
-    <origin xyz="-0.0443 0 0" rpy="0 0 0"/>
-    <parent link="gripper_link"/>
+    <origin xyz="0 0 0" rpy="0 0 0"/>
+    <parent link="end_link"/>
     <child link="gripper_tcp"/>
   </joint>

File: src/rebotarm_moveit_config/config/rebotarm_rs.urdf.xacro (robot description, xacro)
@@ -1,6 +1,6 @@
 <?xml version="1.0"?>
-<robot xmlns:xacro="http://www.ros.org/wiki/xacro" name="rebotarm_rs">
+<robot xmlns:xacro="http://www.ros.org/wiki/xacro" name="ReBot_Arm_RS">
   <xacro:arg name="initial_positions_file" default="$(find rebotarm_moveit_config)/config/initial_positions.yaml"/>
-  <xacro:include filename="$(find rebotarm_bringup)/description/urdf/00-arm-rs_asm-v3.urdf"/>
+  <xacro:include filename="$(find rebotarm_bringup)/description/RS/urdf/ReBot_Arm_RS.urdf"/>
   <xacro:include filename="$(find rebotarm_moveit_config)/config/rebotarm_rs.ros2_control.xacro"/>
   <link name="gripper_tcp"/>
